File: Arquivos EAGLE/fonte.brd (EAGLE design)
At the start: 34 x 57.1 mm, 14 parts, among them Q1 2N3904

Commit message: Add files via upload
Parts:
- C1: value (none) -> 470μ
Changed lines of the file:
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@@
 </autorouter>
 <elements>
-<element name="C1" library="rcl" library_urn="urn:adsk.eagle:library:334" package="E5-10,5" package3d_urn="urn:adsk.eagle:package:23372/2" value="" x="19.05" y="48.26" smashed="yes">
+<element name="C1" library="rcl" library_urn="urn:adsk.eagle:library:334" package="E5-10,5" package3d_urn="urn:adsk.eagle:package:23372/2" value="470μ" x="19.05" y="48.26" smashed="yes">
 <attribute name="NAME" x="23.749" y="51.0032" size="1.27" layer="25" ratio="10"/>
 <attribute name="POPULARITY" value="23" x="57.15" y="41.91" size="1.778" layer="27" display="off"/>
